File: mio.kicad_sch (KiCad schematic)
At the start: 19 parts, among them Q201 MMBT3904, U201 xc7z010clg400, U202 W25Q256FVEI

Commit message: feat: continue ps mio sch design
Parts:
- removed C201, C202: 470n, Capacitor_SMD:C_0402_1005Metric, symbol Device:C
- removed C203: 100n, Capacitor_SMD:C_0402_1005Metric, symbol Device:C
- removed D201: LED, LED_SMD:LED_0603_1608Metric, symbol Device:LED
- removed FB201: 120OHM@100M, Inductor_SMD:L_0603_1608Metric, symbol Device:FerriteBead_Small
- removed Q201: MMBT3904, Package_TO_SOT_SMD:SOT-23, symbol Transistor_BJT:MMBT3904
- removed R201, R205: 1k, Resistor_SMD:R_0402_1005Metric, symbol Device:R
- removed R202, R203: 4k7, Resistor_SMD:R_0402_1005Metric, symbol Device:R
- removed R204: 330R, Resistor_SMD:R_0402_1005Metric, symbol Device:R
- removed R206: 470R, Resistor_SMD:R_0402_1005Metric, symbol Device:R
- removed R207, R208, R209, R210, R211: 20k, Resistor_SMD:R_0402_1005Metric, symbol Device:R
- removed U201: xc7z010clg400, Package_BGA:Xilinx_CLG400, symbol Xilinx7:xc7z010clg400
- removed U202: W25Q256FVEI, Project:IC_W25N04KVZEIU, symbol W25Q256FVEI:W25Q256FVEI
- added C701: 10u, Capacitor_SMD:C_0805_2012Metric, symbol Device:C
- added C702, C703: 100n, Capacitor_SMD:C_0402_1005Metric, symbol Device:C
- added R701, R702, R703: 33R, Resistor_SMD:R_0402_1005Metric, symbol Device:R
- added U201: xc7z010clg400, Package_BGA:Xilinx_CLG400, symbol Xilinx7:xc7z010clg400
- added U701: 33.3333MHz, Oscillator:Oscillator_SMD_SeikoEpson_SG8002CE-4Pin_3.2x2.5mm, symbol Osc33.3333MHz:EPSON_Q33310F700622
Connections:
- net +3V3: now also C701.1, C702.1, C703.1, U201.B6 (VCCO_MIO0_500[2]), U201.D7 (VCCO_MIO0_500[2]), U701.1 (OE), U701.4 (VDD)
- net GND: now also C701.2, C702.2, C703.2, U701.2 (GND)
- net QSPI_CLK: now also R701.1
- net QSPI_CS: now also U201.A7 (PS_MIO1_500)
- net QSPI_D0: now also U201.B8 (PS_MIO2_500)
- net QSPI_D1: now also U201.D6 (PS_MIO3_500)
- net QSPI_D2_PS_MIO4: now also U201.B7 (PS_MIO4_500)
- net QSPI_D3_PS_MIO5: now also U201.A6 (PS_MIO5_500)
- new net: U201.A13 (VCCO_MIO1_501[4]), U201.B16 (VCCO_MIO1_501[4]), U201.D12 (VCCO_MIO1_501[4]), U201.E15 (VCCO_MIO1_501[4])
- new net: R703.2, U201.D14 (PS_MIO40_501)
- new net: R701.2, U201.A5 (PS_MIO6_500)
- new net: R702.2, U201.E7 (PS_CLK_500)
- new net OTG_CLK: U201.A11 (PS_MIO36_501)
- new net OTG_DATA0: U201.A14 (PS_MIO32_501)
- new net OTG_DATA1: U201.D15 (PS_MIO33_501)
- new net OTG_DATA2: U201.A12 (PS_MIO34_501)
- new net OTG_DATA3: U201.F12 (PS_MIO35_501)
- new net OTG_DATA4: U201.C16 (PS_MIO28_501)
- new net OTG_DATA5: U201.A10 (PS_MIO37_501)
- new net OTG_DATA6: U201.E13 (PS_MIO38_501)
- new net OTG_DATA7: U201.C18 (PS_MIO39_501)
- new net OTG_DIR: U201.C13 (PS_MIO29_501)
- new net OTG_NXT: U201.E16 (PS_MIO31_501)
- new net OTG_STP: U201.C15 (PS_MIO30_501)
- new net OTG_nRST: U201.D16 (PS_MIO46_501)
- new net PS_CLK: R702.1, U701.3 (OUT)
- new net PS_SRST_B: U201.B10 (PS_SRST_B_501)
- new net SD_CLK: R703.1
- new net SD_CMD: U201.C17 (PS_MIO41_501)
- new net SD_DATA0: U201.E12 (PS_MIO42_501)
- new net SD_DATA1: U201.A9 (PS_MIO43_501)
- new net SD_DATA2: U201.F13 (PS_MIO44_501)
- new net SD_DATA3: U201.B15 (PS_MIO45_501)
- new net UART_RX: U201.C5 (PS_MIO14_500)
- new net UART_TX: U201.C8 (PS_MIO15_500)
Other:
- note removed: "BOOT OPTION"
