File: ZYNQ-SoM.kicad_sch (KiCad schematic)
At the start: 5 parts, among them U201 xc7z010clg400

Commit message: feat: finish power sch design
Parts:
- renumbered H1 to H101, H2 to H102, H3 to H103, H4 to H104, U201 to U101
Other:
- added sheet POWER (power.kicad_sch)
Changed lines of the file:
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@@
 		(dnp no)
 		(fields_autoplaced yes)
-		(property "Reference" "U201"
+		(property "Reference" "U101"
 			(at 312.42 232.4099 0)
 			(show_name no)
@@
 			(project "ZYNQ-SoM"
 				(path "/49bbd0e9-23a3-4368-9660-7ba6c337a59d"
-					(reference "U201")
+					(reference "U101")
 					(unit 4)
 				)
@@
 		(dnp no)
 		(fields_autoplaced yes)
-		(property "Reference" "U201"
+		(property "Reference" "U101"
 			(at 58.42 350.5199 0)
 			(show_name no)
@@
 			(project "ZYNQ-SoM"
 				(path "/49bbd0e9-23a3-4368-9660-7ba6c337a59d"
-					(reference "U201")
+					(reference "U101")
 					(unit 5)
 				)
@@
 		(dnp no)
 		(fields_autoplaced yes)
-		(property "Reference" "H4"
+		(property "Reference" "H104"
 			(at 264.16 39.3699 0)
 			(show_name no)
@@
 			(project "ZYNQ-SoM"
 				(path "/49bbd0e9-23a3-4368-9660-7ba6c337a59d"
-					(reference "H4")
+					(reference "H104")
 					(unit 1)
 				)
@@
 		(dnp no)
 		(fields_autoplaced yes)
-		(property "Reference" "U201"
+		(property "Reference" "U101"
 			(at 220.98 232.4099 0)
 			(show_name no)
@@
 			(project "ZYNQ-SoM"
 				(path "/49bbd0e9-23a3-4368-9660-7ba6c337a59d"
-					(reference "U201")
+					(reference "U101")
 					(unit 3)
 				)
@@
 		(dnp no)
 		(fields_autoplaced yes)
-		(property "Reference" "H2"
+		(property "Reference" "H102"
 			(at 264.16 26.6699 0)
 			(show_name no)
@@
 			(project "ZYNQ-SoM"
 				(path "/49bbd0e9-23a3-4368-9660-7ba6c337a59d"
-					(reference "H2")
+					(reference "H102")
 					(unit 1)
 				)
@@
 		(dnp no)
 		(fields_autoplaced yes)
-		(property "Reference" "U201"
+		(property "Reference" "U101"
 			(at 346.71 341.6299 0)
 			(show_name no)
@@
 			(project "ZYNQ-SoM"
 				(path "/49bbd0e9-23a3-4368-9660-7ba6c337a59d"
-					(reference "U201")
+					(reference "U101")
 					(unit 8)
 				)
@@
 		(dnp no)
 		(fields_autoplaced yes)
-		(property "Reference" "U201"
+		(property "Reference" "U101"
 			(at 127 170.1799 0)
 			(show_name no)
@@
 			(project "ZYNQ-SoM"
 				(path "/49bbd0e9-23a3-4368-9660-7ba6c337a59d"
-					(reference "U201")
+					(reference "U101")
 					(unit 2)
 				)
@@
 		(dnp no)
 		(fields_autoplaced yes)
-		(property "Reference" "H1"
+		(property "Reference" "H101"
 			(at 264.16 20.3199 0)
 			(show_name no)
@@
 			(project "ZYNQ-SoM"
 				(path "/49bbd0e9-23a3-4368-9660-7ba6c337a59d"
-					(reference "H1")
+					(reference "H101")
 					(unit 1)
 				)
@@
 		(dnp no)
 		(fields_autoplaced yes)
-		(property "Reference" "U201"
+		(property "Reference" "U101"
 			(at 158.75 379.7299 0)
 			(show_name no)
@@
 			(project "ZYNQ-SoM"
 				(path "/49bbd0e9-23a3-4368-9660-7ba6c337a59d"
-					(reference "U201")
+					(reference "U101")
 					(unit 6)
 				)
@@
 		(dnp no)
 		(fields_autoplaced yes)
-		(property "Reference" "H3"
+		(property "Reference" "H103"
 			(at 264.16 33.0199 0)
 			(show_name no)
@@
 			(project "ZYNQ-SoM"
 				(path "/49bbd0e9-23a3-4368-9660-7ba6c337a59d"
-					(reference "H3")
+					(reference "H103")
 					(unit 1)
 				)
@@
 		(dnp no)
 		(fields_autoplaced yes)
-		(property "Reference" "U201"
+		(property "Reference" "U101"
 			(at 360.68 419.0999 0)
 			(show_name no)
@@
 			(project "ZYNQ-SoM"
 				(path "/49bbd0e9-23a3-4368-9660-7ba6c337a59d"
-					(reference "U201")
+					(reference "U101")
 					(unit 9)
 				)
@@
 				)
 			)
+		)
+	)
+	(sheet
+		(at 139.7 50.8)
+		(size 38.1 25.4)
+		(exclude_from_sim no)
+		(in_bom yes)
+		(on_board yes)
+		(dnp no)
+		(fields_autoplaced yes)
+		(stroke
+			(width 0.1524)
+			(type solid)
+		)
+		(fill
+			(color 0 0 0 0)
+		)
+		(property "Sheetname" "POWER"
+			(at 139.7 50.0884 0)
+			(show_name no)
+			(do_not_autoplace no)
+			(effects
+				(font
+					(size 1.27 1.27)
+				)
+				(justify left bottom)
+			)
+		)
+		(property "Sheetfile" "power.kicad_sch"
+			(at 139.7 76.7846 0)
+			(show_name no)
+			(do_not_autoplace no)
+			(effects
+				(font
+					(size 1.27 1.27)
+				)
+				(justify left top)
+			)
+		)
+		(instances
+			(project "ZYNQ-SoM"
+				(path "/49bbd0e9-23a3-4368-9660-7ba6c337a59d"
+					(page "5")
+				)
+			)

Commit message: feat: continue ps mio sch design
Parts:
- removed U101: xc7z010clg400, Package_BGA:Xilinx_CLG400, symbol Xilinx7:xc7z010clg400
Other:
- added sheet PL IO (io.kicad_sch)
- added sheet PS MIO (mio.kicad_sch)
