File: bank0.kicad_sch (KiCad schematic)
At the start: 19 parts, among them Q201 MMBT3904, U201 xc7z010clg400, U202 W25Q256FVEI

Commit message: feat: continue improve sch design
Parts:
- FB201: footprint Inductor_SMD:L_0603_1608Metric -> Inductor_SMD:L_0402_1005Metric
Changed lines of the file:
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@@
 			)
 		)
-		(property "Footprint" "Inductor_SMD:L_0603_1608Metric"
+		(property "Footprint" "Inductor_SMD:L_0402_1005Metric"
 			(at 39.37 76.708 90)
 			(hide yes)
