File: bank0.kicad_sch (KiCad schematic)
At the start: 19 parts, among them Q201 MMBT3904, U201 xc7z010clg400, U202 W25Q256FVEI

Commit message: layout: routing bank 34
Parts:
- removed Q201: MMBT3904, Package_TO_SOT_SMD:SOT-23, symbol Transistor_BJT:MMBT3904
- removed R204: 330R, Resistor_SMD:R_0402_1005Metric, symbol Device:R
- R201: value 1k -> 330R
- R206: value 470R -> 4k7
- U202: footprint Project:IC_W25N04KVZEIU -> Project:SON127P800X600X80-9N-D
Connections:
- net +1V5 is gone; now on net +3V3: R201.1
- net +3V3: now also D201.2 (A); no longer R207.1
- net DONE: now also R201.2; no longer D201.2 (A)
- net GND: now also R205.2, R207.1

Commit message: layout: before rerouting ddr
Changed lines of the file:
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@@
 	)
 	(junction
+		(at 57.15 74.93)
+		(diameter 0)
+		(color 0 0 0 0)
+	)
+	(junction
 		(at 66.04 39.37)
 		(diameter 0)
@@
 	(wire
 		(pts
-			(xy 87.63 74.93) (xy 53.34 74.93)
+			(xy 87.63 74.93) (xy 57.15 74.93)
 		)
 		(stroke
@@
 	(wire
 		(pts
+			(xy 57.15 74.93) (xy 53.34 74.93)
+		)
+		(stroke
+			(width 0)
+			(type default)
+		)
+	)
+	(wire
+		(pts
 			(xy 199.39 66.04) (xy 185.42 66.04)
 		)
@@
 					(unit 1)
 				)
+			)
+		)
+	)
+	(symbol
+		(lib_id "power:PWR_FLAG")
+		(at 57.15 74.93 0)
+		(mirror y)
+		(unit 1)
+		(body_style 1)
+		(exclude_from_sim no)
+		(in_bom yes)
+		(on_board yes)
+		(in_pos_files yes)
+		(dnp no)
+		(property "Reference" "#FLG0201"
+			(at 57.15 73.025 0)
+			(hide yes)
+			(show_name no)
+			(do_not_autoplace no)
+			(effects
+				(font
+					(size 1.27 1.27)
+				)
+			)
+		)
+		(property "Value" "PWR_FLAG"
+			(at 55.88 72.898 0)
+			(show_name no)
+			(do_not_autoplace no)
+			(effects
+				(font
+					(size 1.27 1.27)
+				)
+				(justify left)
+			)
+		)
+		(property "Footprint" ""
+			(at 57.15 74.93 0)
+			(hide yes)
+			(show_name no)
+			(do_not_autoplace no)
+			(effects
+				(font
+					(size 1.27 1.27)
+				)
+			)
+		)
+		(property "Datasheet" ""
+			(at 57.15 74.93 0)
+			(hide yes)
+			(show_name no)
+			(do_not_autoplace no)
+			(effects
+				(font
+					(size 1.27 1.27)
+				)
+			)
+		)
+		(property "Description" "Special symbol for telling ERC where power comes from"
+			(at 57.15 74.93 0)
+			(hide yes)
+			(show_name no)
+			(do_not_autoplace no)
+			(effects
+				(font
+					(size 1.27 1.27)
+				)
+			)
+		)
+		(pin "1"
+		)
+		(instances
+			(project "ZYNQ-SoM"
+				(path "/49bbd0e9-23a3-4368-9660-7ba6c337a59d/2da063c6-0163-4d2d-a242-eeb68f4fd748"
+					(reference "#FLG0201")
+					(unit 1)
+				)
