File: power.kicad_sch (KiCad schematic)
At the start: 94 parts, among them IC501 TPS51206DSQR, U201 xc7z010clg400, U501 TPS62130ARGTR, U502 TPS62130ARGTR, U503 SPX3819M5-L-3-3, U504 TPS62130ARGTR

Commit message: layout: routing bank 34
Parts:
- removed C513, C515, C529, C531: 10u, Capacitor_SMD:C_0805_2012Metric, symbol Device:C
- removed C518: 100u, Capacitor_SMD:C_1206_3216Metric, symbol Device:C
- removed C520, C535: 470n, Capacitor_SMD:C_0402_1005Metric, symbol Device:C
- removed IC501: TPS51206DSQR, Project:SON40P200X200X80-11N, symbol TPS51206DSQR:TPS51206DSQR
Connections:
- net +1V8: no longer C561.1, C567.1, C573.1
- net +3V3: now also C561.1, C567.1, C573.1
- net 1V8_SW: now reaches L503.1, U504.1 (SW_1), U504.2 (SW_2), U504.3 (SW_3)
- net 1V5_SW: now reaches L502.1, U502.1 (SW_1), U502.2 (SW_2), U502.3 (SW_3)
- net 1V0_SW: now reaches L501.1, U501.1 (SW_1), U501.2 (SW_2), U501.3 (SW_3)
Other:
- note removed: "VCCIO 13"
- moved on the sheet: L501, L502, L503

Commit message: layout: before rerouting ddr
Parts:
- removed C537, C557: 4u7, Capacitor_SMD:C_0603_1608Metric, symbol Device:C
- C507, C540: footprint Capacitor_SMD:C_0805_2012Metric -> Capacitor_SMD:C_0603_1608Metric
- U503: PACKAGE (none) -> SOT-23-5
Other:
- moved on the sheet: C507, C508, C539, C542, C543, C544, C548, C549, C554, C555, C558, C559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
