File: ddr3.kicad_sch (KiCad schematic)
At the start: 49 parts, among them U201 xc7z010clg400, U301 MT41K256M16TW-107_P

Commit message: layout: routing bank 34
Parts:
- removed C315: 10u, Capacitor_SMD:C_0805_2012Metric, symbol Device:C
- removed C317, C321, C322: 100n, Capacitor_SMD:C_0402_1005Metric, symbol Device:C
- removed R308, R309, R310, R311, R312, R313, R314, R315, R316, R317, R318, R319, R320, R321, R322, R323, R324, R325, R326, R327, R328, R329, R330: 40R2, Resistor_SMD:R_0402_1005Metric, symbol Device:R
- added R303: 80R6, Resistor_SMD:R_0402_1005Metric, symbol Device:R
- C311: value 10n -> 100n
- R307: value 40R2 -> 80R6
Connections:
- net +DDRVTT is gone; now on net +VTTREF: R307.2
- net VTTREF is gone; now on net +VTTREF: C311.1, C313.1, U201.H6 (PS_DDR_VREF0_502), U201.P6 (PS_DDR_VREF1_502)
- net +1V5: now also R307.1
- net +VTTREF: now also R303.1
- net DDR_A0: no longer R307.1
- net DDR_CLK_N: now also U201.M2 (PS_DDR_CKN_502); no longer U201.L2 (PS_DDR_CKP_502)
- net DDR_CLK_P: now also U201.L2 (PS_DDR_CKP_502); no longer U201.M2 (PS_DDR_CKN_502)
- net DDR_D0: now also U301.F7 (DQ1); no longer U301.G2 (DQ6)
- net DDR_D1: now also U301.G2 (DQ6); no longer U301.F2 (DQ2)
- net DDR_D10: now also U301.C3 (DQ9); no longer U301.A3 (DQ15)
- net DDR_D11: now also U301.C2 (DQ11); no longer U301.D7 (DQ8)
- net DDR_D12: now also U301.D7 (DQ8); no longer U301.C3 (DQ9)
- net DDR_D13: now also U301.A7 (DQ12); no longer U301.B8 (DQ14)
- net DDR_D14: now also U301.B8 (DQ14); no longer U301.A7 (DQ12)
- net DDR_D2: now also U301.F2 (DQ2); no longer U301.E3 (DQ0)
- net DDR_D4: now also U301.H7 (DQ7); no longer U301.H8 (DQ5)
- net DDR_D5: now also U301.F8 (DQ3); no longer U301.F7 (DQ1)
- net DDR_D6: now also U301.E3 (DQ0); no longer U301.F8 (DQ3)
- net DDR_D7: now also U301.H8 (DQ5); no longer U301.H7 (DQ7)
- net DDR_D8: now also U301.A3 (DQ15); no longer U301.C2 (DQ11)
- net GND: now also R303.2
Other:
- moved on the sheet: C313
