File: connector.kicad_sch (KiCad schematic)
At the start: 2 parts, among them J401 AXK500137YG, J402 AXK500137YG

Commit message: layout: add bank 34 pl pair
Connections:
- net PL_B34_IO0 is gone; now on net PL_B34_IO20_N: J401.53
- net PL_B34_IO23_P is gone; now on net PL_B34_IO20_P: J401.55
- net +5V: now also J401.13, J401.14, J401.15, J401.16
- net GND: no longer J401.15, J401.16
- net PL_B34_IO12_N: now also J401.67; no longer J401.24
- net PL_B34_IO12_P: now also J401.65; no longer J401.26
- net PL_B34_IO13_N: now also J401.43; no longer J401.38
- net PL_B34_IO13_P: now also J401.41; no longer J401.36
- net PL_B34_IO14_N: now also J401.35; no longer J401.67
- net PL_B34_IO14_P: now also J401.37; no longer J401.65
- net PL_B34_IO20_N: no longer J401.32
- net PL_B34_IO20_P: no longer J401.30
- net PL_B34_IO22_N: now also J401.38; no longer J401.20
- net PL_B34_IO22_P: now also J401.36; no longer J401.18
- net PL_B34_IO4_N: now also J401.59; no longer J401.61
- net PL_B34_IO4_P: now also J401.61; no longer J401.59
- net PL_B34_IO23_N renamed PL_B34_IO24_N
- net PL_B34_IO25 renamed PL_B34_IO24_P
- no-connect marks 12 -> 4
